File: CLKGEN.kicad_sch (KiCad schematic)
At the start: 16 parts

Commit message: annotated and packages defined
Parts:
- C13, C14, C15: renamed from C?; footprint (none) -> Capacitor_SMD:C_0805_2012Metric
- R47, R48, R49, R50, R51, R52, R53, R55, R56: renamed from R?; footprint (none) -> Resistor_SMD:R_0805_2012Metric
- R54: renamed from R?; value DNP -> 0R-DNP; footprint (none) -> Resistor_SMD:R_0805_2012Metric
- Y1: renamed from Y?; value DNP (25/27 MHz 3225) -> 25/27MHz-3225-DNP; footprint (none) -> Crystal:Crystal_SMD_3225-4Pin_3.2x2.5mm_HandSoldering
- gave numbers to parts that had none: 2
Connections:
- no-connect marks 0 -> 1
Other:
- company: (none) -> papamidas DM1CR
- title: (none) -> H7DDCADC

Commit message: placement 80 percent
Parts:
- added R86: 0R, Resistor_SMD:R_0805_2012Metric, symbol Device:R
Connections:
- net CLK1: now also R86.2; no longer U14.9 (CLK1)
- new net: R86.1, U14.9 (CLK1)
Changed lines of the file:
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@@
     (stroke (width 0) (type default) (color 0 0 0 0))
   )
-  (wire (pts (xy 177.8 118.11) (xy 241.3 118.11))
+  (wire (pts (xy 177.8 118.11) (xy 182.88 118.11))
+    (stroke (width 0) (type default) (color 0 0 0 0))
+  )
+  (wire (pts (xy 190.5 118.11) (xy 241.3 118.11))
     (stroke (width 0) (type default) (color 0 0 0 0))
   )
@@
     (pin "1")
   )
+  (symbol (lib_id "Device:R") (at 186.69 118.11 90) (unit 1)
+    (in_bom yes) (on_board yes)
+    (property "Reference" "R86" (id 0) (at 186.69 120.65 90))
+    (property "Value" "0R" (id 1) (at 191.77 120.65 90))
+    (property "Footprint" "Resistor_SMD:R_0805_2012Metric" (id 2) (at 186.69 119.888 90)
+      (effects (font (size 1.27 1.27)) hide)
+    )
+    (property "Datasheet" "~" (id 3) (at 186.69 118.11 0)
+      (effects (font (size 1.27 1.27)) hide)
+    )
+    (pin "1")
+    (pin "2")
+  )
 )
