File: POWER.kicad_sch (KiCad schematic)
At the start: 16 parts

Commit message: annotated and packages defined
Parts:
- C20, C21, C22, C23, C24, C25, C26: renamed from C?; footprint (none) -> Capacitor_SMD:C_0805_2012Metric
- FB1: renamed from FB?; footprint (none) -> Resistor_SMD:R_0805_2012Metric
- R81, R82, R83: renamed from R?; footprint (none) -> Resistor_SMD:R_0805_2012Metric
- R84, R85: renamed from R?; value DNP -> 0R-DNP; footprint (none) -> Resistor_SMD:R_0805_2012Metric
- gave numbers to parts that had none: 3
Other:
- company: (none) -> papamidas DM1CR
- title: (none) -> H7DDCADC

Commit message: routing in progress 1
Parts:
- added C29, C30: 1uF, Capacitor_SMD:C_0805_2012Metric, symbol Device:C_Small
- added FB2: Ferrite_0805, Resistor_SMD:R_0805_2012Metric, symbol Device:FerriteBead_Small
Connections:
- net GND: now also C29.2, C30.2
- net VIN: now also C29.1, FB2.1; no longer C20.1, C21.1, C22.1, FB1.1, R81.1, R82.1, R83.1, U23.1 (VIN), U24.1 (VIN), U25.1 (VIN)
- new net +3V3F: C20.1, C21.1, C22.1, C30.1, FB1.1, FB2.2, R81.1, R82.1, R83.1, U23.1 (VIN), U24.1 (VIN), U25.1 (VIN)
Changed lines of the file:
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@@
   (junction (at 119.38 85.09) (diameter 0) (color 0 0 0 0)
   )
+  (junction (at 45.72 48.26) (diameter 0) (color 0 0 0 0)
+  )
+  (junction (at 72.39 48.26) (diameter 0) (color 0 0 0 0)
+  )
   (junction (at 92.71 48.26) (diameter 0) (color 0 0 0 0)
   )
@@
   (junction (at 128.27 97.79) (diameter 0) (color 0 0 0 0)
   )
+  (junction (at 92.71 25.4) (diameter 0) (color 0 0 0 0)
+  )
   (junction (at 106.68 85.09) (diameter 0) (color 0 0 0 0)
   )
@@
     (stroke (width 0) (type default) (color 0 0 0 0))
   )
+  (wire (pts (xy 45.72 54.61) (xy 45.72 55.88))
+    (stroke (width 0) (type default) (color 0 0 0 0))
+  )
   (wire (pts (xy 127 74.93) (xy 127 87.63))
     (stroke (width 0) (type default) (color 0 0 0 0))
@@
     (stroke (width 0) (type default) (color 0 0 0 0))
   )
+  (wire (pts (xy 72.39 48.26) (xy 92.71 48.26))
+    (stroke (width 0) (type default) (color 0 0 0 0))
+  )
   (wire (pts (xy 119.38 58.42) (xy 119.38 60.96))
     (stroke (width 0) (type default) (color 0 0 0 0))
@@
     (stroke (width 0) (type default) (color 0 0 0 0))
   )
+  (wire (pts (xy 72.39 48.26) (xy 72.39 49.53))
+    (stroke (width 0) (type default) (color 0 0 0 0))
+  )
   (wire (pts (xy 142.24 25.4) (xy 162.56 25.4))
     (stroke (width 0) (type default) (color 0 0 0 0))
   )
-  (wire (pts (xy 87.63 48.26) (xy 92.71 48.26))
+  (wire (pts (xy 39.37 48.26) (xy 45.72 48.26))
     (stroke (width 0) (type default) (color 0 0 0 0))
   )
@@
     (stroke (width 0) (type default) (color 0 0 0 0))
   )
+  (wire (pts (xy 45.72 48.26) (xy 45.72 49.53))
+    (stroke (width 0) (type default) (color 0 0 0 0))
+  )
   (wire (pts (xy 92.71 48.26) (xy 106.68 48.26))
     (stroke (width 0) (type default) (color 0 0 0 0))
@@
     (stroke (width 0) (type default) (color 0 0 0 0))
   )
+  (wire (pts (xy 92.71 15.24) (xy 92.71 25.4))
+    (stroke (width 0) (type default) (color 0 0 0 0))
+  )
   (wire (pts (xy 106.68 48.26) (xy 106.68 49.53))
     (stroke (width 0) (type default) (color 0 0 0 0))
   )
+  (wire (pts (xy 205.74 15.24) (xy 92.71 15.24))
+    (stroke (width 0) (type default) (color 0 0 0 0))
+  )
   (wire (pts (xy 107.95 132.08) (xy 107.95 133.35))
     (stroke (width 0) (type default) (color 0 0 0 0))
@@
     (stroke (width 0) (type default) (color 0 0 0 0))
   )
+  (wire (pts (xy 63.5 48.26) (xy 72.39 48.26))
+    (stroke (width 0) (type default) (color 0 0 0 0))
+  )
   (wire (pts (xy 119.38 48.26) (xy 119.38 50.8))
     (stroke (width 0) (type default) (color 0 0 0 0))
@@
     (stroke (width 0) (type default) (color 0 0 0 0))
   )
+  (wire (pts (xy 45.72 48.26) (xy 58.42 48.26))
+    (stroke (width 0) (type default) (color 0 0 0 0))
+  )
   (wire (pts (xy 167.64 132.08) (xy 167.64 133.35))
     (stroke (width 0) (type default) (color 0 0 0 0))
   )
   (wire (pts (xy 138.43 58.42) (xy 138.43 59.69))
+    (stroke (width 0) (type default) (color 0 0 0 0))
+  )
+  (wire (pts (xy 72.39 54.61) (xy 72.39 55.88))
     (stroke (width 0) (type default) (color 0 0 0 0))
   )
@@
     (effects (font (size 1.27 1.27)) (justify left))
   )
+  (hierarchical_label "+3V3F" (shape output) (at 205.74 15.24 0)
+    (effects (font (size 1.27 1.27)) (justify left))
+  )
   (hierarchical_label "ENA18" (shape input) (at 106.68 97.79 180)
     (effects (font (size 1.27 1.27)) (justify right))
   )
-  (hierarchical_label "VIN" (shape input) (at 87.63 48.26 180)
+  (hierarchical_label "VIN" (shape input) (at 39.37 48.26 180)
     (effects (font (size 1.27 1.27)) (justify right))
   )
@@
     (pin "2")
   )
+  (symbol (lib_id "power:GND") (at 45.72 55.88 0) (unit 1)
+    (in_bom yes) (on_board yes)
+    (property "Reference" "#PWR096" (id 0) (at 45.72 62.23 0)
+      (effects (font (size 1.27 1.27)) hide)
+    )
+    (property "Value" "GND" (id 1) (at 49.53 57.15 0))
+    (property "Footprint" "" (id 2) (at 45.72 55.88 0)
+      (effects (font (size 1.27 1.27)) hide)
+    )
+    (property "Datasheet" "" (id 3) (at 45.72 55.88 0)
+      (effects (font (size 1.27 1.27)) hide)
+    )
+    (pin "1")
+  )
   (symbol (lib_id "Device:C_Small") (at 167.64 129.54 0) (unit 1)
     (in_bom yes) (on_board yes) (fields_autoplaced)
@@
     (pin "1")
   )
+  (symbol (lib_id "Device:FerriteBead_Small") (at 60.96 48.26 90) (unit 1)
+    (in_bom yes) (on_board yes) (fields_autoplaced)
+    (property "Reference" "FB2" (id 0) (at 60.9219 41.91 90))
+    (property "Value" "Ferrite_0805" (id 1) (at 60.9219 44.45 90))
+    (property "Footprint" "Resistor_SMD:R_0805_2012Metric" (id 2) (at 60.96 50.038 90)
+      (effects (font (size 1.27 1.27)) hide)
+    )
+    (property "Datasheet" "~" (id 3) (at 60.96 48.26 0)
+      (effects (font (size 1.27 1.27)) hide)
+    )
+    (pin "1")
+    (pin "2")
+  )
   (symbol (lib_id "power:GND") (at 166.37 55.88 0) (unit 1)
     (in_bom yes) (on_board yes)
@@
     (pin "1")
   )
+  (symbol (lib_id "Device:C_Small") (at 45.72 52.07 0) (unit 1)
+    (in_bom yes) (on_board yes) (fields_autoplaced)
+    (property "Reference" "C29" (id 0) (at 48.26 50.8062 0)
+      (effects (font (size 1.27 1.27)) (justify left))
+    )
+    (property "Value" "1uF" (id 1) (at 48.26 53.3462 0)
+      (effects (font (size 1.27 1.27)) (justify left))
+    )
+    (property "Footprint" "Capacitor_SMD:C_0805_2012Metric" (id 2) (at 45.72 52.07 0)
+      (effects (font (size 1.27 1.27)) hide)
+    )
+    (property "Datasheet" "~" (id 3) (at 45.72 52.07 0)
+      (effects (font (size 1.27 1.27)) hide)
+    )
+    (pin "1")
+    (pin "2")
+  )
+  (symbol (lib_id "Device:C_Small") (at 72.39 52.07 0) (unit 1)
+    (in_bom yes) (on_board yes) (fields_autoplaced)
+    (property "Reference" "C30" (id 0) (at 74.93 50.8062 0)
+      (effects (font (size 1.27 1.27)) (justify left))
+    )
+    (property "Value" "1uF" (id 1) (at 74.93 53.3462 0)
+      (effects (font (size 1.27 1.27)) (justify left))
+    )
+    (property "Footprint" "Capacitor_SMD:C_0805_2012Metric" (id 2) (at 72.39 52.07 0)
+      (effects (font (size 1.27 1.27)) hide)
+    )
+    (property "Datasheet" "~" (id 3) (at 72.39 52.07 0)
+      (effects (font (size 1.27 1.27)) hide)
+    )
+    (pin "1")
+    (pin "2")
+  )
   (symbol (lib_id "Regulator_Linear:AP2127K-1.8") (at 138.43 50.8 0) (unit 1)
     (in_bom yes) (on_board yes) (fields_autoplaced)
@@
       (effects (font (size 1.27 1.27)) hide)
     )
+    (pin "1")
+  )
+  (symbol (lib_id "power:GND") (at 72.39 55.88 0) (unit 1)
+    (in_bom yes) (on_board yes)
+    (property "Reference" "#PWR097" (id 0) (at 72.39 62.23 0)
+      (effects (font (size 1.27 1.27)) hide)
+    )
+    (property "Value" "GND" (id 1) (at 76.2 57.15 0))
+    (property "Footprint" "" (id 2) (at 72.39 55.88 0)
+      (effects (font (size 1.27 1.27)) hide)
+    )
+    (property "Datasheet" "" (id 3) (at 72.39 55.88 0)
+      (effects (font (size 1.27 1.27)) hide)
+    )
