File: ADC.kicad_sch (KiCad schematic)
At the start: 32 parts

Commit message: annotated and packages defined
Parts:
- C1, C2: renamed from C?; footprint (none) -> Capacitor_SMD:C_0805_2012Metric
- J5: renamed from J?; value HDR4_2 -> HDR2x4; footprint (none) -> Connector_PinHeader_2.54mm:PinHeader_2x04_P2.54mm_Vertical; Field4 (none) -> CLK_AUX
- R10, R11, R14, R16, R17, R18, R7, R9: renamed from R?; value DNP -> 200-DNP; footprint (none) -> Resistor_SMD:R_0805_2012Metric
- R12, R13, R15, R19, R20, R21, R8: renamed from R?; footprint (none) -> Resistor_SMD:R_0805_2012Metric
- U10: renamed from U?; value 74AUC2G79 -> 74AUC2G79DCT; footprint (none) -> Package_SO:MSOP-8_3x3mm_P0.65mm
- U10, U9: renamed from U?; value (none) -> 74AUC2G79DCT; footprint (none) -> Package_SO:MSOP-8_3x3mm_P0.65mm
- U11: renamed from U?; value (none) -> 74AUC1G08DBV; footprint (none) -> Package_TO_SOT_SMD:SOT-23-5
- U12: renamed from U?; value ~ -> 74AUC1G74DCT; footprint (none) -> Package_SO:VSSOP-8_2.4x2.1mm_P0.5mm
- U3: renamed from U?; footprint (none) -> Package_DFN_QFN:UQFN-40-1EP_5x5mm_P0.4mm_EP3.8x3.8mm_ThermalVias
- U4, U6: renamed from U?; value ~ -> 74AUC2G34DBV; footprint (none) -> Package_TO_SOT_SMD:SOT-23-6_Handsoldering
- U5, U6: renamed from U?; value 74AUC2G34 -> 74AUC2G34DBV; footprint (none) -> Package_TO_SOT_SMD:SOT-23-6_Handsoldering
- U8: renamed from U?; value 74AUC1G74 -> 74AUC1G74DCT; footprint (none) -> Package_SO:VSSOP-8_2.4x2.1mm_P0.5mm
Connections:
- net DCLK_IN_D3: no longer J5.5 (Pin_5)
- new net DCLK_IN_ADC: J5.5 (Pin_5)
- no-connect marks 8 -> 10
Other:
- company: (none) -> papamidas DM1CR
- title: (none) -> H7DDCADC

Commit message: placement_in_progress 1
Connections:
- net DA1_FCLK_ADC: now also U4.3; no longer U4.1
- net DA6_ADC: now also U4.1; no longer U4.3
- net at U11.2, U8.2 (D): now also U4.4; no longer U4.6
- net at U9.2 (D): now also U4.6; no longer U4.4
Other:
- note added: "Output decoupling resistors connected to all ADC pins, even to NC pins, for easier later upgrade to ADC3664 etc."
- note added: "TI suffix DBV = SOT23 TI suffix DCK = SC70 TI suffix DCT = SM8 (SSOP, 0.65 mm pitch) TI suffix DCU = VSSOP (MSOP, 0.5 mm pitch)"
- note removed: "SN74AUC2G34DBV (= SOT23) SN74AUC1G08DBV (= SOT23) SN74AUC1G74DCT (= SM8) SN74AUC1G74DCU (= VSSOP) SN74AUC2G79DCT (= SM8) SN74AUC2G79DCU (=VSSOP)"
Changed lines of the file:
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@@
     (stroke (width 0) (type default) (color 0 0 0 0))
   )
-  (text "SN74AUC2G34DBV (= SOT23)\nSN74AUC1G08DBV (= SOT23)\nSN74AUC1G74DCT (= SM8)\nSN74AUC1G74DCU (= VSSOP)\nSN74AUC2G79DCT (= SM8)\nSN74AUC2G79DCU (=VSSOP)\n"
-    (at 119.38 26.67 0)
+  (text "TI suffix DBV = SOT23\nTI suffix DCK = SC70\nTI suffix DCT = SM8 (SSOP, 0.65 mm pitch)\nTI suffix DCU = VSSOP (MSOP, 0.5 mm pitch)"
+    (at 185.42 22.86 0)
+    (effects (font (size 1.27 1.27)) (justify left bottom))
+  )
+  (text "Output decoupling resistors connected to all ADC pins,\neven to NC pins, for easier later upgrade to ADC3664 etc."
+    (at 104.14 45.72 0)
     (effects (font (size 1.27 1.27)) (justify left bottom))
   )
@@
     (pin "1")
   )
-  (symbol (lib_id "74xGxx:74AUC2G34") (at 160.02 69.85 0) (unit 2)
+  (symbol (lib_id "74xGxx:74AUC2G34") (at 160.02 69.85 0) (unit 1)
     (in_bom yes) (on_board yes)
     (property "Reference" "U4" (id 0) (at 163.83 66.04 0))
@@
     (pin "1")
   )
-  (symbol (lib_id "74xGxx:74AUC2G34") (at 160.02 57.15 0) (unit 1)
+  (symbol (lib_id "74xGxx:74AUC2G34") (at 160.02 57.15 0) (unit 2)
     (in_bom yes) (on_board yes)
     (property "Reference" "U4" (id 0) (at 163.83 53.34 0))

Commit message: placement 80 percent
Parts:
- R10, R11, R12, R13, R14, R15, R16, R17, R18, R19, R20, R21, R7, R8, R9: footprint Resistor_SMD:R_0805_2012Metric -> Resistor_SMD:R_0402_1005Metric_Pad0.72x0.64mm_HandSolder
Changed lines of the file:
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@@
     (property "Reference" "R14" (id 0) (at 113.03 73.66 90))
     (property "Value" "200-DNP" (id 1) (at 127 73.66 90))
-    (property "Footprint" "Resistor_SMD:R_0805_2012Metric" (id 2) (at 118.11 76.708 90)
+    (property "Footprint" "Resistor_SMD:R_0402_1005Metric_Pad0.72x0.64mm_HandSolder" (id 2) (at 118.11 76.708 90)
       (effects (font (size 1.27 1.27)) hide)
     )
@@
     (property "Reference" "R9" (id 0) (at 113.03 58.42 90))
     (property "Value" "200-DNP" (id 1) (at 127 58.42 90))
-    (property "Footprint" "Resistor_SMD:R_0805_2012Metric" (id 2) (at 118.11 61.468 90)
+    (property "Footprint" "Resistor_SMD:R_0402_1005Metric_Pad0.72x0.64mm_HandSolder" (id 2) (at 118.11 61.468 90)
       (effects (font (size 1.27 1.27)) hide)
     )
@@
     (property "Reference" "R17" (id 0) (at 113.03 81.28 90))
     (property "Value" "200-DNP" (id 1) (at 127 81.28 90))
-    (property "Footprint" "Resistor_SMD:R_0805_2012Metric" (id 2) (at 118.11 84.328 90)
+    (property "Footprint" "Resistor_SMD:R_0402_1005Metric_Pad0.72x0.64mm_HandSolder" (id 2) (at 118.11 84.328 90)
       (effects (font (size 1.27 1.27)) hide)
     )
@@
     (property "Reference" "R11" (id 0) (at 113.03 63.5 90))
     (property "Value" "200-DNP" (id 1) (at 127 63.5 90))
-    (property "Footprint" "Resistor_SMD:R_0805_2012Metric" (id 2) (at 118.11 66.548 90)
+    (property "Footprint" "Resistor_SMD:R_0402_1005Metric_Pad0.72x0.64mm_HandSolder" (id 2) (at 118.11 66.548 90)
       (effects (font (size 1.27 1.27)) hide)
     )
@@
     (property "Reference" "R20" (id 0) (at 113.03 88.9 90))
     (property "Value" "200" (id 1) (at 124.46 88.9 90))
-    (property "Footprint" "Resistor_SMD:R_0805_2012Metric" (id 2) (at 118.11 88.392 90)
+    (property "Footprint" "Resistor_SMD:R_0402_1005Metric_Pad0.72x0.64mm_HandSolder" (id 2) (at 118.11 88.392 90)
       (effects (font (size 1.27 1.27)) hide)
     )
@@
     (property "Reference" "R18" (id 0) (at 113.03 83.82 90))
     (property "Value" "200-DNP" (id 1) (at 127 83.82 90))
-    (property "Footprint" "Resistor_SMD:R_0805_2012Metric" (id 2) (at 118.11 86.868 90)
+    (property "Footprint" "Resistor_SMD:R_0402_1005Metric_Pad0.72x0.64mm_HandSolder" (id 2) (at 118.11 86.868 90)
       (effects (font (size 1.27 1.27)) hide)
     )
@@
     (property "Reference" "R13" (id 0) (at 113.03 68.58 90))
     (property "Value" "200" (id 1) (at 124.46 68.58 90))
-    (property "Footprint" "Resistor_SMD:R_0805_2012Metric" (id 2) (at 118.11 68.072 90)
+    (property "Footprint" "Resistor_SMD:R_0402_1005Metric_Pad0.72x0.64mm_HandSolder" (id 2) (at 118.11 68.072 90)
       (effects (font (size 1.27 1.27)) hide)
     )
@@
     (property "Reference" "R15" (id 0) (at 113.03 76.2 90))
     (property "Value" "200" (id 1) (at 124.46 76.2 90))
-    (property "Footprint" "Resistor_SMD:R_0805_2012Metric" (id 2) (at 118.11 79.248 90)
+    (property "Footprint" "Resistor_SMD:R_0402_1005Metric_Pad0.72x0.64mm_HandSolder" (id 2) (at 118.11 79.248 90)
       (effects (font (size 1.27 1.27)) hide)
     )
@@
     (property "Reference" "R16" (id 0) (at 113.03 78.74 90))
     (property "Value" "200-DNP" (id 1) (at 127 78.74 90))
-    (property "Footprint" "Resistor_SMD:R_0805_2012Metric" (id 2) (at 118.11 81.788 90)
+    (property "Footprint" "Resistor_SMD:R_0402_1005Metric_Pad0.72x0.64mm_HandSolder" (id 2) (at 118.11 81.788 90)
       (effects (font (size 1.27 1.27)) hide)
     )
@@
     (property "Reference" "R12" (id 0) (at 113.03 66.04 90))
     (property "Value" "200" (id 1) (at 124.46 66.04 90))
-    (property "Footprint" "Resistor_SMD:R_0805_2012Metric" (id 2) (at 118.11 69.088 90)
+    (property "Footprint" "Resistor_SMD:R_0402_1005Metric_Pad0.72x0.64mm_HandSolder" (id 2) (at 118.11 69.088 90)
       (effects (font (size 1.27 1.27)) hide)
     )
@@
     (property "Reference" "R19" (id 0) (at 113.03 86.36 90))
     (property "Value" "200" (id 1) (at 124.46 86.36 90))
-    (property "Footprint" "Resistor_SMD:R_0805_2012Metric" (id 2) (at 118.11 85.852 90)
+    (property "Footprint" "Resistor_SMD:R_0402_1005Metric_Pad0.72x0.64mm_HandSolder" (id 2) (at 118.11 85.852 90)
       (effects (font (size 1.27 1.27)) hide)
     )
@@
     (property "Reference" "R8" (id 0) (at 113.03 55.88 90))
     (property "Value" "200" (id 1) (at 124.46 55.88 90))
-    (property "Footprint" "Resistor_SMD:R_0805_2012Metric" (id 2) (at 118.11 58.928 90)
+    (property "Footprint" "Resistor_SMD:R_0402_1005Metric_Pad0.72x0.64mm_HandSolder" (id 2) (at 118.11 58.928 90)
       (effects (font (size 1.27 1.27)) hide)
     )
@@
     (property "Reference" "R10" (id 0) (at 113.03 60.96 90))
     (property "Value" "200-DNP" (id 1) (at 127 60.96 90))
-    (property "Footprint" "Resistor_SMD:R_0805_2012Metric" (id 2) (at 118.11 64.008 90)
+    (property "Footprint" "Resistor_SMD:R_0402_1005Metric_Pad0.72x0.64mm_HandSolder" (id 2) (at 118.11 64.008 90)
       (effects (font (size 1.27 1.27)) hide)
     )
@@
     (property "Reference" "R7" (id 0) (at 113.03 53.34 90))
     (property "Value" "200-DNP" (id 1) (at 127 53.34 90))
-    (property "Footprint" "Resistor_SMD:R_0805_2012Metric" (id 2) (at 118.11 56.388 90)
+    (property "Footprint" "Resistor_SMD:R_0402_1005Metric_Pad0.72x0.64mm_HandSolder" (id 2) (at 118.11 56.388 90)
       (effects (font (size 1.27 1.27)) hide)
     )
@@
     (property "Reference" "R21" (id 0) (at 113.03 93.98 90))
     (property "Value" "200" (id 1) (at 124.46 93.98 90))
-    (property "Footprint" "Resistor_SMD:R_0805_2012Metric" (id 2) (at 118.11 97.028 90)
-      (effects (font (size 1.27 1.27)) hide)
-    )
+    (property "Footprint" "Resistor_SMD:R_0402_1005Metric_Pad0.72x0.64mm_HandSolder" (id 2) (at 118.11 97.028 90)
+      (effects (font (size 1.27 1.27)) hide)
+    )

Commit message: routing in progress 1
Parts:
- removed J5: HDR2x4, Connector_PinHeader_2.54mm:PinHeader_2x04_P2.54mm_Vertical, symbol Connector_Generic:Conn_02x04_Odd_Even
- removed U3: ADC3660IRSBT, Package_DFN_QFN:UQFN-40-1EP_5x5mm_P0.4mm_EP3.8x3.8mm_ThermalVias, symbol DM1CR_Library:ADC3660IRSBT
- added C31, C32, C33, C34, C35: 100n, Capacitor_SMD:C_0402_1005Metric_Pad0.74x0.62mm_HandSolder, symbol Device:C_Small
- added TP10: CLKP_ADC, TestPoint:TestPoint_THTPad_D1.5mm_Drill0.7mm, symbol Connector:TestPoint
- added TP11: CLKN_ADC, TestPoint:TestPoint_THTPad_D1.5mm_Drill0.7mm, symbol Connector:TestPoint
- added TP12: DCLK_IN_D3, TestPoint:TestPoint_THTPad_D1.5mm_Drill0.7mm, symbol Connector:TestPoint
- added TP13: DCLK_ADC, TestPoint:TestPoint_THTPad_D1.5mm_Drill0.7mm, symbol Connector:TestPoint
- added TP14, TP15, TP16, TP17, TP18: GND, TestPoint:TestPoint_THTPad_D1.5mm_Drill0.7mm, symbol Connector:TestPoint
- added U3: ADC3660IRSBT, Package_DFN_QFN:QFN-40-1EP_5x5mm_P0.4mm_EP3.6x3.6mm, symbol DM1CR_Library_loc:ADC3660IRSBT
Connections:
- net AIN_N: now also U3.13 (AINM)
- net AIN_P: now also U3.12 (AINP)
- net AVDD: now also C33.1, C34.1, C35.1, U3.15 (AVDD), U3.36 (AVDD), U3.5 (AVDD)
- net BIN_N: now also U3.38 (BINM)
- net BIN_P: now also U3.39 (BINP)
- net CLKN_ADC: now also TP11.1, U3.7 (CLKM)
- net CLKP_ADC: now also TP10.1, U3.6 (CLKP)
- net DCLK_ADC: now also TP13.1
- net DCLK_IN_D3: now also TP12.1
- net GND: now also C31.2, C32.2, C33.2, C34.2, C35.2, TP14.1, TP15.1, TP16.1, TP17.1, TP18.1, U3.11 (GND), U3.14 (GND), U3.26 (IOGND), U3.3 (REFGND), U3.37 (GND), U3.40 (GND), U3.41 (GND_PAD)
- net IOVDD: now also C31.1, C32.1, U3.21 (IOVDD), U3.30 (IOVDD)
- net PDN_SYNC: now also U3.1 (PDN/SYNC)
- net REFBUF: now also U3.4 (REFBUF)
- net RESET: now also U3.9 (RESET)
- net SCLK: now also U3.35 (SCLK)
- net SDIO: now also U3.10 (SDIO)
- net SEN: now also U3.16 (/SEN)
- net VCM: now also U3.8 (VCM)
- net VREF: now also U3.2 (VREF)
- net at R14.1: now also U3.34 (NC)
- net at R7.1: now also U3.17 (NC)
- net at R8.1: now also U3.18 (FCLK)
- net at R9.1: now also U3.19 (NC)
- net at R10.1: now also U3.20 (NC)
- net at R11.1: now also U3.22 (NC)
- net at R12.1: now also U3.23 (DA5)
- net at R13.2: now also U3.24 (DA6)
- net at R21.1: now also U3.25 (DCLK)
- net at R20.2: now also U3.27 (DB6)
- net at R19.2: now also U3.28 (DB5)
- net at R18.1: now also U3.29 (NC)
- net at R17.1: now also U3.31 (NC)
- net at R16.1: now also U3.32 (NC)
- net at R15.1: now also U3.33 (DCLKIN)
Other:
- moved on the sheet: C1, C2, R21

Commit message: routing in progress 2
Parts:
- added C41, C42, C43, C44, C45, C46, C47, C48: 100n, Capacitor_SMD:C_0402_1005Metric_Pad0.74x0.62mm_HandSolder, symbol Device:C_Small
- U3: footprint Package_DFN_QFN:QFN-40-1EP_5x5mm_P0.4mm_EP3.6x3.6mm -> Package_DFN_QFN:UQFN-40-1EP_5x5mm_P0.4mm_EP3.8x3.8mm_ThermalVias
Connections:
- net GND: now also C41.2, C42.2, C43.2, C44.2, C45.2, C46.2, C47.2, C48.2
- net IOVDD: now also C41.1, C42.1, C43.1, C44.1, C45.1, C46.1, C47.1, C48.1
