File: H7DDCADC.kicad_sch (KiCad schematic)
At the start: 14 parts

Commit message: annotated and packages defined
Parts:
- added TP3: ENA18, TestPoint:TestPoint_THTPad_D1.5mm_Drill0.7mm, symbol Connector:TestPoint
- added TP4: DA5, TestPoint:TestPoint_THTPad_D1.5mm_Drill0.7mm, symbol Connector:TestPoint
- added TP5: DB5, TestPoint:TestPoint_THTPad_D1.5mm_Drill0.7mm, symbol Connector:TestPoint
- added TP6: NSS_D, TestPoint:TestPoint_THTPad_D1.5mm_Drill0.7mm, symbol Connector:TestPoint
- added TP7: DCK_B, TestPoint:TestPoint_THTPad_D1.5mm_Drill0.7mm, symbol Connector:TestPoint
- added TP8: DA6_D, TestPoint:TestPoint_THTPad_D1.5mm_Drill0.7mm, symbol Connector:TestPoint
- added TP9: DB6_D, TestPoint:TestPoint_THTPad_D1.5mm_Drill0.7mm, symbol Connector:TestPoint
- J1: renamed from J?; value EXT_CLK -> U.FL-DNP; footprint (none) -> Connector_Coaxial:U.FL_Hirose_U.FL-R-SMT-1_Vertical; Field4 (none) -> EXT_CLK
- J2: renamed from J?; value CH_A -> SMA; footprint (none) -> Connector_Coaxial:SMA_Wurth_60312002114503_Vertical; Field4 (none) -> CH A IN
- J3: renamed from J?; value CH_B -> SMA; footprint (none) -> Connector_Coaxial:SMA_Wurth_60312002114503_Vertical; Field4 (none) -> CH B IN
- J4: renamed from J?; value EXT_VREF -> HDR2; footprint (none) -> Connector_PinHeader_2.54mm:PinHeader_1x02_P2.54mm_Vertical; Field4 (none) -> EXT_VREF
- R1, R4, R5: renamed from R?; value DNP -> 0R-DNP; footprint (none) -> Resistor_SMD:R_0805_2012Metric
- R2, R3, R6: renamed from R?; footprint (none) -> Resistor_SMD:R_0805_2012Metric
- TP1: renamed from TP?; footprint (none) -> TestPoint:TestPoint_THTPad_D1.5mm_Drill0.7mm
- TP2: renamed from TP?; value DCLK_B2 -> DCK_B2; footprint (none) -> TestPoint:TestPoint_THTPad_D1.5mm_Drill0.7mm
- U1, U2: renamed from U?; value (none) -> 74AUC1G74DCT; footprint (none) -> Package_SO:VSSOP-8_2.4x2.1mm_P0.5mm
Connections:
- net ADC/DA5_ADC: now also TP4.1
- net ADC/DA6_DELAYED: now also TP8.1
- net ADC/DB5_ADC: now also TP5.1
- net ADC/DB6_DELAYED: now also TP9.1
- net ADC/DCLK_BUFD: now also TP7.1
- net ADC/NSS_DELAYED: now also TP6.1
- net Power/ENA18: now also TP3.1
- no-connect marks 0 -> 5
Other:
- company: (none) -> papamidas DM1CR
- title: (none) -> H7DDCADC

Commit message: placement_in_progress 1
Connections:
- net ADC/DA6_DELAYED renamed DA6_D_50
- net ADC/DB6_DELAYED renamed DB6_D_50
- net ADC/DCLK_BUFD renamed DCK_B_50
- net ADC/NSS_DELAYED renamed NSS_D_50
- net ADCINP_A/GNDI renamed GNDI_A
- net ADCINP_A/IN renamed IN_A_50
- net ADCINP_B/GNDI renamed GNDI_B
- net ADCINP_B/IN renamed IN_B_50
Other:
- note added: "TI suffix DCT = SM8 (SSOP, 0.65 mm pitch)"
Changed lines of the file:
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@@
+    (stroke (width 0) (type default) (color 0 0 0 0))
+  )
+  (wire (pts (xy 204.47 128.27) (xy 207.01 128.27))
     (stroke (width 0) (type default) (color 0 0 0 0))
   )
@@
     (stroke (width 0) (type default) (color 0 0 0 0))
   )
+  (wire (pts (xy 204.47 139.7) (xy 207.01 139.7))
+    (stroke (width 0) (type default) (color 0 0 0 0))
+  )
   (wire (pts (xy 144.78 30.48) (xy 161.29 30.48))
     (stroke (width 0) (type default) (color 0 0 0 0))
@@
     (stroke (width 0) (type default) (color 0 0 0 0))
   )
+  (wire (pts (xy 204.47 134.62) (xy 207.01 134.62))
+    (stroke (width 0) (type default) (color 0 0 0 0))
+  )
   (wire (pts (xy 256.54 88.9) (xy 256.54 128.27))
     (stroke (width 0) (type default) (color 0 0 0 0))
@@
   )
   (wire (pts (xy 242.57 101.6) (xy 247.65 101.6))
+    (stroke (width 0) (type default) (color 0 0 0 0))
+  )
+  (wire (pts (xy 204.47 144.78) (xy 207.01 144.78))
     (stroke (width 0) (type default) (color 0 0 0 0))
   )
@@
     (effects (font (size 1.27 1.27)) (justify left bottom))
   )
+  (text "TI suffix DCT = SM8 (SSOP, 0.65 mm pitch)\n" (at 147.32 144.78 0)
+    (effects (font (size 1.27 1.27)) (justify left bottom))
+  )
   (text "ADC" (at 123.19 68.58 0)
     (effects (font (size 1.27 1.27)) (justify left bottom))
   )
+  (label "DCK_B_50" (at 149.86 55.88 0)
+    (effects (font (size 1.27 1.27)) (justify left bottom))
+  )
   (label "ECLK_IN" (at 48.26 97.79 0)
     (effects (font (size 1.27 1.27)) (justify left bottom))
   )
+  (label "IN_A_50" (at 50.8 29.21 0)
+    (effects (font (size 1.27 1.27)) (justify left bottom))
+  )
+  (label "SPI2_SCK_50" (at 191.77 53.34 0)
+    (effects (font (size 1.27 1.27)) (justify left bottom))
+  )
+  (label "SP3_NNS_50" (at 191.77 33.02 0)
+    (effects (font (size 1.27 1.27)) (justify left bottom))
+  )
   (label "CLKN_IN" (at 116.84 113.03 0)
     (effects (font (size 1.27 1.27)) (justify left bottom))
   )
+  (label "SPI3_MOSI_50" (at 191.77 48.26 0)
+    (effects (font (size 1.27 1.27)) (justify left bottom))
+  )
+  (label "DA6_D_50" (at 149.86 38.1 0)
+    (effects (font (size 1.27 1.27)) (justify left bottom))
+  )
+  (label "SPI2_NSS_50" (at 191.77 29.21 0)
+    (effects (font (size 1.27 1.27)) (justify left bottom))
+  )
+  (label "NSS_D_50" (at 149.86 30.48 0)
+    (effects (font (size 1.27 1.27)) (justify left bottom))
+  )
   (label "DCLK_IN" (at 99.06 76.2 0)
     (effects (font (size 1.27 1.27)) (justify left bottom))
@@
     (effects (font (size 1.27 1.27)) (justify left bottom))
   )
+  (label "GNDI_A" (at 52.07 34.29 0)
+    (effects (font (size 1.27 1.27)) (justify left bottom))
+  )
+  (label "IN_B_50" (at 50.8 49.53 0)
+    (effects (font (size 1.27 1.27)) (justify left bottom))
+  )
   (label "ECLK_IN" (at 172.72 113.03 0)
     (effects (font (size 1.27 1.27)) (justify left bottom))
   )
+  (label "SPI2_MOSI_50" (at 191.77 38.1 0)
+    (effects (font (size 1.27 1.27)) (justify left bottom))
+  )
   (label "CLK_P_IN" (at 99.06 81.28 0)
     (effects (font (size 1.27 1.27)) (justify left bottom))
   )
+  (label "SPI3_SCK_50" (at 191.77 57.15 0)
+    (effects (font (size 1.27 1.27)) (justify left bottom))
+  )
   (label "DCLK_IN" (at 115.57 132.08 0)
+    (effects (font (size 1.27 1.27)) (justify left bottom))
+  )
+  (label "DB6_D_50" (at 149.86 48.26 0)
+    (effects (font (size 1.27 1.27)) (justify left bottom))
+  )
+  (label "GNDI_B" (at 52.07 54.61 0)
     (effects (font (size 1.27 1.27)) (justify left bottom))
   )
@@
     (pin "1")
   )
-  (symbol (lib_id "DM1CR_Library:IOVDD") (at 207.01 139.7 90) (unit 1)
-    (in_bom yes) (on_board yes)
-    (property "Reference" "#PWR031" (id 0) (at 210.82 139.7 0)
-      (effects (font (size 1.27 1.27)) hide)
-    )
-    (property "Value" "IOVDD" (id 1) (at 200.66 139.7 90))
-    (property "Footprint" "" (id 2) (at 207.01 139.7 0)
-      (effects (font (size 1.27 1.27)) hide)
-    )
-    (property "Datasheet" "" (id 3) (at 207.01 139.7 0)
+  (symbol (lib_id "DM1CR_Library:IOVDD") (at 204.47 139.7 90) (unit 1)
+    (in_bom yes) (on_board yes)
+    (property "Reference" "#PWR031" (id 0) (at 208.28 139.7 0)
+      (effects (font (size 1.27 1.27)) hide)
+    )
+    (property "Value" "IOVDD" (id 1) (at 198.12 139.7 90))
+    (property "Footprint" "" (id 2) (at 204.47 139.7 0)
+      (effects (font (size 1.27 1.27)) hide)
+    )
+    (property "Datasheet" "" (id 3) (at 204.47 139.7 0)
       (effects (font (size 1.27 1.27)) hide)
     )
@@
     (pin "2")
   )
-  (symbol (lib_id "DM1CR_Library:AVDD") (at 207.01 134.62 90) (unit 1)
-    (in_bom yes) (on_board yes)
-    (property "Reference" "#PWR030" (id 0) (at 210.82 134.62 0)
-      (effects (font (size 1.27 1.27)) hide)
-    )
-    (property "Value" "AVDD" (id 1) (at 200.66 134.62 90))
-    (property "Footprint" "" (id 2) (at 207.01 134.62 0)
-      (effects (font (size 1.27 1.27)) hide)
-    )
-    (property "Datasheet" "" (id 3) (at 207.01 134.62 0)
+  (symbol (lib_id "DM1CR_Library:AVDD") (at 204.47 134.62 90) (unit 1)
+    (in_bom yes) (on_board yes)
+    (property "Reference" "#PWR030" (id 0) (at 208.28 134.62 0)
+      (effects (font (size 1.27 1.27)) hide)
+    )
+    (property "Value" "AVDD" (id 1) (at 198.12 134.62 90))
+    (property "Footprint" "" (id 2) (at 204.47 134.62 0)
+      (effects (font (size 1.27 1.27)) hide)
+    )
+    (property "Datasheet" "" (id 3) (at 204.47 134.62 0)
       (effects (font (size 1.27 1.27)) hide)
     )
@@
     (pin "1")
   )
-  (symbol (lib_id "power:+1V8") (at 207.01 144.78 90) (unit 1)
-    (in_bom yes) (on_board yes)
-    (property "Reference" "#PWR032" (id 0) (at 210.82 144.78 0)
-      (effects (font (size 1.27 1.27)) hide)
-    )
-    (property "Value" "+1V8" (id 1) (at 198.12 144.78 90)
-      (effects (font (size 1.27 1.27)) (justify right))
-    )
-    (property "Footprint" "" (id 2) (at 207.01 144.78 0)
-      (effects (font (size 1.27 1.27)) hide)
-    )
-    (property "Datasheet" "" (id 3) (at 207.01 144.78 0)
+  (symbol (lib_id "power:+1V8") (at 204.47 144.78 90) (unit 1)
+    (in_bom yes) (on_board yes)
+    (property "Reference" "#PWR032" (id 0) (at 208.28 144.78 0)
+      (effects (font (size 1.27 1.27)) hide)
+    )
+    (property "Value" "+1V8" (id 1) (at 195.58 144.78 90)
+      (effects (font (size 1.27 1.27)) (justify right))
+    )
+    (property "Footprint" "" (id 2) (at 204.47 144.78 0)
+      (effects (font (size 1.27 1.27)) hide)
+    )
+    (property "Datasheet" "" (id 3) (at 204.47 144.78 0)
       (effects (font (size 1.27 1.27)) hide)
     )
@@
     (pin "1")
   )
-  (symbol (lib_id "power:+3.3VA") (at 207.01 128.27 90) (unit 1)
-    (in_bom yes) (on_board yes)
-    (property "Reference" "#PWR029" (id 0) (at 210.82 128.27 0)
-      (effects (font (size 1.27 1.27)) hide)
-    )
-    (property "Value" "+3.3VA" (id 1) (at 196.85 128.27 90)
-      (effects (font (size 1.27 1.27)) (justify right))
-    )
-    (property "Footprint" "" (id 2) (at 207.01 128.27 0)
-      (effects (font (size 1.27 1.27)) hide)
-    )
-    (property "Datasheet" "" (id 3) (at 207.01 128.27 0)
+  (symbol (lib_id "power:+3.3VA") (at 204.47 128.27 90) (unit 1)
+    (in_bom yes) (on_board yes)
+    (property "Reference" "#PWR029" (id 0) (at 208.28 128.27 0)
+      (effects (font (size 1.27 1.27)) hide)
+    )
+    (property "Value" "+3.3VA" (id 1) (at 194.31 128.27 90)
+      (effects (font (size 1.27 1.27)) (justify right))
+    )
+    (property "Footprint" "" (id 2) (at 204.47 128.27 0)
+      (effects (font (size 1.27 1.27)) hide)
+    )
+    (property "Datasheet" "" (id 3) (at 204.47 128.27 0)
       (effects (font (size 1.27 1.27)) hide)
     )
@@
       (reference "U3") (unit 1) (value "ADC3660IRSBT") (footprint "Package_DFN_QFN:UQFN-40-1EP_5x5mm_P0.4mm_EP3.8x3.8mm_ThermalVias")
     )
+    (path "/9b65c9d0-858c-4826-94e3-1e53a6bb86da/a66f84b0-1aeb-4b9f-8582-c67d153aed9e"
+      (reference "U4") (unit 1) (value "74AUC2G34DBV") (footprint "Package_TO_SOT_SMD:SOT-23-6_Handsoldering")
+    )
     (path "/9b65c9d0-858c-4826-94e3-1e53a6bb86da/ba57cea8-5b60-4446-bb14-67c5d94248d7"
-      (reference "U4") (unit 1) (value "74AUC2G34DBV") (footprint "Package_TO_SOT_SMD:SOT-23-6_Handsoldering")
-    )
-    (path "/9b65c9d0-858c-4826-94e3-1e53a6bb86da/a66f84b0-1aeb-4b9f-8582-c67d153aed9e"
       (reference "U4") (unit 2) (value "74AUC2G34DBV") (footprint "Package_TO_SOT_SMD:SOT-23-6_Handsoldering")
     )

Commit message: routing in progress 1
Parts:
- added R87, R88: 0R, Resistor_SMD:R_0805_2012Metric, symbol Device:R
Connections:
- net GND: now also R87.1, R88.1
- net GNDI_A: now also R87.2
- net GNDI_B: now also R88.2
Other:
- sheet ADCTRANSL ports: added VSUP; removed VCC
- sheet MCU ports: added VCC_1T97; removed none
- sheet Power ports: added +3V3F; removed none

Commit message: routing in progress 2
Parts:
- added C39, C40: 100n, Capacitor_SMD:C_0402_1005Metric_Pad0.74x0.62mm_HandSolder, symbol Device:C_Small
- added R89, R90: 0R-DNP, Resistor_SMD:R_0805_2012Metric, symbol Device:R
Connections:
- net CLKGEN/EXT_IN: now also R90.2; no longer R1.2
- net ECLK_IN: now also R89.1; no longer R4.1
- net GND: now also C39.2, C40.2
- net IOVDD: now also C39.1, C40.1
- new net CLKN_ECKL_50: R4.1, R89.2
- new net EXT_ECLK_50: R1.2, R90.1
Other:
- moved on the sheet: R1
